Commit message: save big data files to git lfs

File: urdfs/quadrotor.urdf.xacro (robot description, xacro)
@@ -2,5 +2,5 @@
 <robot name="quadrotor" xmlns:xacro="http://www.ros.org/wiki/xacro">
     <xacro:property name="M_PI" value="3.1415926535897931" />
-    <xacro:property name="M_PI/2" value="1.5707963267945" />
+    <xacro:property name="M_PI_2" value="1.5707963267945" />
     <!-- Included URDF Files -->
     <xacro:include filename="./quadrotor_base.urdf.xacro" />
@@ -10,5 +10,5 @@
     <xacro:include filename="$(find hector_sensors_description)/urdf/hokuyo_utm30lx.urdf.xacro" />
     <xacro:hokuyo_utm30lx name="laser0" parent="base_link" ros_topic="scan" update_rate="40" ray_count="1081" min_angle="-90" max_angle="90">
-      <origin xyz="0.0 0.0 0.15" rpy="-${M_PI} -${M_PI/2} ${M_PI/2}"/>
+      <origin xyz="0.0 0.0 0.15" rpy="-${M_PI} -${M_PI_2} ${M_PI_2}"/>
     </xacro:hokuyo_utm30lx>
 </robot>
