Commit message: test

File: urdfs/quadrotor_base.urdf.xacro (robot description, xacro)
@@ -31,4 +31,18 @@
             </collision>
         </link>
+        <gazebo reference="base_link">
+					<sensor name="quad_contact_sensor" type="contact">
+						<always_on>true</always_on>
+						<update_rate>30.0</update_rate>
+						<visualize>true</visualize>
+						<contact>
+							<collision>collision_collision</collision>
+						</contact>
+						<plugin name="gazebo_ros_bumper_plugin" filename="libgazebo_ros_bumper.so">
+							<bumperTopicName>gazebo_ros_bumper</bumperTopicName>
+							<frameName>world</frameName>
+						</plugin>
+					</sensor>
+				</gazebo>
     <!-- Hokuyo UTM-30LX sensor -->
     <!--<xacro:include filename="$(find hector_sensors_description)/urdf/hokuyo_utm30lx.urdf.xacro" />-->
