Commit message: (1) Add new methods for fixing the NAN output of PPO, but the effect is not tested. The methods are: <1> keep detecting observation in both env and reset if there is NAN among it. <2> clip gradient norm when necessary, otherwise keep old unclipped style, if NAN happens, use 'continue' to go to next iteration.
(2) Try different action transformation in simple car example.

(3) Note the consistency of angle definition between gazebo and brs_engine. Have been Fixed.

File: urdfs/dubins_car.urdf.xacro (robot description, xacro)
@@ -1,9 +1,22 @@
 <?xml version="1.0"?>
-<robot name="dubins_car" xmlns:xacro="http://www.ros.org/wiki/xacro">
+<!--
+    - Base      : kobuki
+    - Stacks    : hexagons
+    - Sensors   : None
+-->
+<robot name="turtlebot" xmlns:xacro="http://ros.org/wiki/xacro">
     <xacro:property name="M_PI" value="3.1415926535897931" />
     <xacro:property name="M_PI_2" value="1.5707963267945" />
-    <!-- Included URDF Files -->
-    <xacro:include filename="dubins_car_base.urdf.xacro" />
-    <!-- Instantiate quadrotor_base_macro once (has no parameters atm) -->
-    <xacro:dubins_car_base_macro />
+  <xacro:include filename="$(find turtlebot_description)/urdf/turtlebot_common_library.urdf.xacro" />
+  <xacro:include filename="$(find kobuki_description)/urdf/kobuki.urdf.xacro" />
+  <xacro:include filename="$(find turtlebot_description)/urdf/stacks/hexagons.urdf.xacro"/>
+  <!-- <xacro:include filename="$(find turtlebot_description)/urdf/sensors/asus_xtion_pro.urdf.xacro"/> -->
+  <kobuki/>
+  <stack_hexagons                 parent="base_link"/>
+  <!-- <sensor_asus_xtion_pro          parent="base_link"/> -->
+    <!-- Hokuyo UTM-30LX sensor -->
+    <xacro:include filename="$(find hector_sensors_description)/urdf/hokuyo_utm30lx.urdf.xacro" />
+    <xacro:hokuyo_utm30lx name="laser0" parent="base_link" ros_topic="scan" update_rate="40" ray_count="1081" min_angle="-90" max_angle="90">
+      <origin xyz="0.0 0.0 0.45" rpy="0 0 0"/>
+    </xacro:hokuyo_utm30lx>
 </robot>
